File: cape/WillowCape_v1.brd (EAGLE design)
At the start: 5.7 x 54.6 mm, 69 parts, among them U1 SN74LV245, U2 SN74LV245, U3 SN74LV245, U4 SN74LV245, U5 SN74LV245, U6 SN74LV245

Commit message: Done with v1 of control box. Motion sensors aren't connected yet but there are placeholders
Parts:
- moved C3 376.1 mm to (55.9, 78.2)
- moved C1 355.6 mm to (60.8, 52.5), turned to 180 degrees
- moved C2 340.3 mm to (36.4, 53.2), turned to 270 degrees
- moved C6 325.8 mm to (15.5, 36.3), flipped to the bottom, turned to 180 degrees
- moved R48 19.9 mm to (25.0, 49.0), flipped to the bottom, turned to 180 degrees
- moved R47 19.7 mm to (25.0, 46.7), flipped to the bottom, turned to 180 degrees
- moved R41 18.0 mm to (25.0, 33.1), flipped to the bottom, turned to 180 degrees
- moved R42 17.8 mm to (25.0, 35.4), flipped to the bottom, turned to 180 degrees
- moved R46 8.64 mm to (25.0, 44.6), flipped to the bottom, turned to 180 degrees
- moved C5 6.41 mm to (55.9, 11.0)
- moved R43 6.31 mm to (25.0, 37.7), flipped to the bottom, turned to 180 degrees
- moved R45 4.70 mm to (25.0, 42.3), flipped to the bottom, turned to 180 degrees
- moved C4 3.81 mm to (36.8, 25.4), turned to 90 degrees
- moved R6 3.56 mm to (62.1, 49.3)
- moved R8 3.56 mm to (62.2, 46.1)
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Connections:
- removed net N$1: JP1.P1, JP2.P1, JP3.P1, JP4.P1, JP5.P1, JP6.P1, JP7.P1, JP8.P1
- removed net N$10: JP1.P6, JP2.P6, JP3.P6, JP4.P6, JP5.P6, JP6.P6, JP7.P6, JP8.P6
- removed net N$11: JP1.P8, JP2.P8, JP3.P8, JP4.P8, JP5.P8, JP6.P8, JP7.P8, JP8.P8
- removed net N$111: R1.2, R17.2, R25.2, R33.2, R9.2
- removed net N$112: R10.2, R18.2, R2.2, R26.2, R34.2
- removed net N$113: R11.2, R19.2, R27.2, R3.2, R35.2
- removed net N$114: R12.2, R20.2, R28.2, R36.2, R4.2
- removed net N$115: R13.2, R21.2, R29.2, R37.2, R5.2
- removed net N$116: R14.2, R22.2, R30.2, R38.2, R6.2
- removed net N$117: R15.2, R23.2, R31.2, R39.2, R7.2
- removed net N$118: R16.2, R24.2, R32.2, R40.2, R8.2
- removed net N$12: JP1.P10, JP2.P10, JP3.P10, JP4.P10, JP5.P10, JP6.P10, JP7.P10, JP8.P10
- removed net N$13: JP1.P12, JP2.P12, JP3.P12, JP4.P12, JP5.P12, JP6.P12, JP7.P12, JP8.P12
- removed net N$14: JP1.P14, JP2.P14, JP3.P14, JP4.P14, JP5.P14, JP6.P14, JP7.P14, JP8.P14
- removed net N$2: JP1.P3, JP2.P3, JP3.P3, JP4.P3, JP5.P3, JP6.P3, JP7.P3, JP8.P3
- removed net N$3: JP1.P5, JP2.P5, JP3.P5, JP4.P5, JP5.P5, JP6.P5, JP7.P5, JP8.P5
- removed net N$4: JP1.P7, JP2.P7, JP3.P7, JP4.P7, JP5.P7, JP6.P7, JP7.P7, JP8.P7
- removed net N$5: JP1.P9, JP2.P9, JP3.P9, JP4.P9, JP5.P9, JP6.P9, JP7.P9, JP8.P9
- removed net N$6: JP1.P11, JP2.P11, JP3.P11, JP4.P11, JP5.P11, JP6.P11, JP7.P11, JP8.P11
- removed net N$7: JP1.P13, JP2.P13, JP3.P13, JP4.P13, JP5.P13, JP6.P13, JP7.P13, JP8.P13
- removed net N$9: JP1.P4, JP2.P4, JP3.P4, JP4.P4, JP5.P4, JP6.P4, JP7.P4, JP8.P4
- new net M1S1: JP1.P4, R18.2
- new net M1S2: JP1.P6, R17.2
- new net M1S3: JP1.P8, R19.2
- new net M1S4: JP1.P10, R20.2
- new net M1S5: JP1.P12, R21.2
- new net M2S1: JP2.P4, R24.2
- new net M2S2: JP2.P6, R23.2
- new net M2S3: JP2.P8, R22.2
- new net M2S4: JP2.P10, R4.2
- new net M2S5: JP2.P12, R3.2
- new net M3S1: JP3.P4, R2.2
- new net M3S2: JP3.P6, R1.2
- new net M3S3: JP3.P8, R5.2
- new net M3S4: JP3.P10, R6.2
- new net M3S5: JP3.P12, R7.2
- new net M4S1: JP4.P4, R9.2
- new net M4S2: JP4.P6, R8.2
- new net M4S3: JP4.P8, R10.2
- new net M4S4: JP4.P10, R11.2
- new net M4S5: JP4.P12, R12.2
- new net M5S1: JP5.P4, R16.2
- new net M5S2: JP5.P6, R15.2
- new net M5S3: JP5.P8, R14.2
- new net M5S4: JP5.P10, R13.2
- new net M5S5: JP5.P12, R25.2
- new net M6S1: JP6.P4, R32.2
- new net M6S2: JP6.P6, R28.2
- new net M6S3: JP6.P8, R27.2
- new net M6S4: JP6.P10, R26.2
- new net M6S5: JP6.P12, R31.2
- new net M7S1: JP7.P4, R33.2
- new net M7S2: JP7.P6, R34.2
- new net M7S3: JP7.P8, R35.2
- new net M7S4: JP7.P10, R29.2
- new net M7S5: JP7.P12, R30.2
- new net M8S1: JP8.P4, R39.2
- new net M8S2: JP8.P6, R40.2
- new net M8S3: JP8.P8, R38.2
- new net M8S4: JP8.P10, R37.2
- new net M8S5: JP8.P12, R36.2
- net 5V: now also U2.1, U2.20
- net CLK0_1: now also JP8.P2; no longer JP2.P2
- net CLK0_2: now also JP7.P2; no longer JP1.P2
- net CLK0_3: now also JP6.P2; no longer JP3.P2
- net CLK0_4: now also JP5.P2; no longer JP4.P2
- net CLK1_1: now also JP4.P2; no longer JP5.P2
- net CLK1_2: now also JP3.P2; no longer JP6.P2
- net CLK1_3: now also JP2.P2; no longer JP7.P2
- net CLK1_4: now also JP1.P2; no longer JP8.P2
- net GND: now also JP1.P1, JP1.P11, JP1.P13, JP1.P14, JP1.P3, JP1.P5, JP1.P7, JP1.P9, JP2.P1, JP2.P11, JP2.P13, JP2.P14, JP2.P3, JP2.P5, JP2.P7, JP2.P9, JP3.P1, JP3.P11, JP3.P13, JP3.P14, JP3.P3, JP3.P5, JP3.P7, JP3.P9, JP4.P1, JP4.P11, JP4.P13, JP4.P14, JP4.P3, JP4.P5, JP4.P7, JP4.P9, JP5.P1, JP5.P11, JP5.P13, JP5.P14, JP5.P3, JP5.P5, JP5.P7, JP5.P9, JP6.P1, JP6.P11, JP6.P13, JP6.P14, JP6.P3, JP6.P5, JP6.P7, JP6.P9, JP7.P1, JP7.P11, JP7.P13, JP7.P14, JP7.P3, JP7.P5, JP7.P7, JP7.P9, JP8.P1, JP8.P11, JP8.P13, JP8.P14, JP8.P3, JP8.P5, JP8.P7, JP8.P9
Routing:
- net CLK1_4: track 0.00 -> 65.0 mm
- net CLK1_3: track 0.00 -> 61.8 mm
- net CLK1_2: track 0.00 -> 58.5 mm
- net CLK1_1: track 0.00 -> 55.2 mm
- net CLK0_4: track 0.00 -> 55.1 mm
- net M4S4: track 0.00 -> 54.3 mm
- net M4S5: track 0.00 -> 53.5 mm
- net M5S4: track 0.00 -> 52.9 mm
- net M4S3: track 0.00 -> 46.9 mm
- net M5S2: track 0.00 -> 46.5 mm
- net M5S3: track 0.00 -> 46.3 mm
- net M4S1: track 0.00 -> 46.0 mm
- net M6S5: track 0.00 -> 40.6 mm
- net M5S5: track 0.00 -> 40.6 mm
- net M5S1: track 0.00 -> 39.9 mm
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Other:
- board size 5.7 x 54.6 mm -> 100.3 x 80 mm
- board text added: "5V"
- board text added: "Designed by Shlomo Zippel"
- board text added: "GND"
- board text added: "M1"
- board text added: "M2"
- board text added: "M3"
- board text added: "M4"
- board text added: "M5"
- board text added: "M6"
- board text added: "M7"
- board text added: "M8"
- board text added: "Willow Tree Control Box"
- board text added: "v1"
